File: misc/schematics/midimagic.kicad_sch (KiCad schematic)
At the start: 96 parts, among them J1 Port0_analog, J10 MIDI_Thru_DIN-5_180degree, J11 SSD1306_Display_128x64px, J12 Port7_digital, J13 Port6_digital, J14 Port5_digital, J15 Port4_digital, J16 Port3_digital, J17 Port2_digital, J18 Port1_digital, J19 Port0_digital, J2 Port1_analog, J20 From PSU, J3 Port2_analog, J4 Port3_analog, J5 Port4_analog, J6 Port5_analog, J7 Port6_analog, J8 Port7_analog, J9 MIDI_In_DIN-5_180degree, Q1 2N7000, Q2 BS250, SW1 RotaryEncoder, U1 STM32F103C8Tx, U10 LM4040LP-2.5, U11 Generic_fixed_voltage_regulat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, U2 AD57x4_on_adaptor, U3 AD57x4_on_adaptor, U4 TL074, U5 TL074, U6 H11L1, U7 TL071, U8 TL074, U9 TL074

Commit message: switch to dedicated external eeprom, refactor archive handling
Parts:
- added U12: 93LCxxC, symbol Memory_EEPROM:93LCxxC
Connections:
- net +3V3: now also U12.8 (VCC)
- net GNDA: now also U12.5 (GND), U12.6 (ORG)
- net at U1.12 (PA2): now also U12.2 (SCLK)
- net at U1.13 (PA3): now also U12.1 (CS)
- net at U1.18 (PB0): now also U12.3 (DI)
- net at U1.19 (PB1): now also U12.4 (DO)
- no-connect marks 31 -> 27

Commit message: update schematic
Parts:
- added C28: 100 nF, symbol Device:C_Small
- added R35: 1K, symbol Device:R_Small
Connections:
- net GNDA: now also C28.1
- net at U1.28 (PB15): now also C28.2, R35.1; no longer SW1.S1
- new net: R35.2, SW1.S1
Other:
- note added: "If the EEPROM has a Program Enable (PE) Pin tie it to VCC"
